File: watch pcb/watch pcb.kicad_pcb (KiCad board)
At the start: 2 copper layers, 44 x 44 mm, 10 parts, among them J1 DISPLAY, J2 BATTERY, J3 WIRELESS_RECEIVER, J4 VIBRATING MOTOR, J5 ACCELEROMETER, Q1 2N2222, SW1 POWER SWITCH, U1 XIAO-ESP32-C6-SMD

Commit message: final
Parts:
- added REF**: MountingHole_3.2mm_M3, MountingHole:MountingHole_3.2mm_M3, F.Cu at (131.0, 57.0)
